Commit message: Rebase from 'upstream'

File: playground_kobuki/easynav_playground_kobuki_description/urdf/kobuki.urdf.xacro (robot description, xacro)
@@ -9,5 +9,5 @@
   <xacro:arg name="camera" default="false" />
   <xacro:arg name="structure" default="false" />
-  <xacro:arg name="lidar_range" default="3.0" />
+  <xacro:arg name="lidar_range" default="12.0" />
   <!-- Namespace will be applied to all TF frames and topics.
        This is required if multiple robots are launched at the same time.

File: playground_kobuki/easynav_playground_kobuki_description/urdf/kobuki_base.urdf.xacro (robot description, xacro)
@@ -58,5 +58,5 @@
       <parent link="$(arg namespace)base_link"/>
       <child link="$(arg namespace)wheel_left_link"/>
-      <origin xyz="0.00 ${0.25/2} 0.0250" rpy="${-M_PI/2} 0 0"/>
+      <origin xyz="0.00 ${0.23/2} 0.0250" rpy="${-M_PI/2} 0 0"/>
       <axis xyz="0 0 1"/>
     </joint>
@@ -85,5 +85,5 @@
       <parent link="$(arg namespace)base_link"/>
       <child link="$(arg namespace)wheel_right_link"/>
-      <origin xyz="0.00 -${0.25/2} 0.0250" rpy="${-M_PI/2} 0 0"/>
+      <origin xyz="0.00 -${0.23/2} 0.0250" rpy="${-M_PI/2} 0 0"/>
       <axis xyz="0 0 1"/>
     </joint>

File: playground_kobuki/easynav_playground_kobuki_description/urdf/kobuki_gazebo.urdf.xacro (robot description, xacro)
@@ -1,10 +1,10 @@
 <?xml version="1.0" ?>
 <robot name="kobuki_gazebo" xmlns:xacro="http://ros.org/wiki/xacro">
-  <xacro:macro name="kobuki_gazebo" params="lidar camera namespace tf_namespace lidar_range:=3.0">
+  <xacro:macro name="kobuki_gazebo" params="lidar camera namespace tf_namespace lidar_range:=12.0">
     <gazebo>
       <plugin filename="gz-sim-diff-drive-system" name="gz::sim::systems::DiffDrive">
         <left_joint>$(arg namespace)wheel_left_joint</left_joint>
         <right_joint>$(arg namespace)wheel_right_joint</right_joint>
-        <wheel_separation>0.223087</wheel_separation>
+        <wheel_separation>0.230</wheel_separation>
         <wheel_radius>0.035</wheel_radius>
         <max_linear_acceleration>1.0</max_linear_acceleration>
